File: sImCP.kicad_pcb (KiCad board)
At the start: 2 copper layers, 155.6 x 140 mm, 79 parts, among them J1 AVR-ISP-6, SW1 RESET, SW2 BOOT, U1 ATmega328P-AU, Y1 16MHz

Commit message: update rocker switch 3dmodel
Parts:
- renumbered H6 to M2, H5 to M2, H4 to M3, H3 to M3, H2 to M3, H1 to M3
Changed lines of the file:
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@@
     (tags "mounting hole 2.2mm m2 din965")
     (attr virtual)
-    (fp_text reference H6 (at 0 -2.9) (layer F.SilkS)
+    (fp_text reference M2 (at 0 -2.9) (layer F.SilkS)
       (effects (font (size 1 1) (thickness 0.15)))
     )
@@
     (tags "mounting hole 2.2mm m2 din965")
     (attr virtual)
-    (fp_text reference H5 (at 0 -2.9) (layer F.SilkS)
+    (fp_text reference M2 (at 0 -2.9) (layer F.SilkS)
       (effects (font (size 1 1) (thickness 0.15)))
     )
@@
     (tags "mounting hole 3.2mm m3 iso7380")
     (attr virtual)
-    (fp_text reference H4 (at 0 -3.85) (layer F.SilkS)
+    (fp_text reference M3 (at 0 -3.85) (layer F.SilkS)
       (effects (font (size 1 1) (thickness 0.15)))
     )
@@
     (tags "mounting hole 3.2mm m3 iso7380")
     (attr virtual)
-    (fp_text reference H3 (at 0 -3.85) (layer F.SilkS)
+    (fp_text reference M3 (at 0 -3.85) (layer F.SilkS)
       (effects (font (size 1 1) (thickness 0.15)))
     )
@@
     (tags "mounting hole 3.2mm m3 iso7380")
     (attr virtual)
-    (fp_text reference H2 (at 0 -3.85) (layer F.SilkS)
+    (fp_text reference M3 (at 0 4.28) (layer F.SilkS)
       (effects (font (size 1 1) (thickness 0.15)))
     )
@@
     (tags "mounting hole 3.2mm m3 iso7380")
     (attr virtual)
-    (fp_text reference H1 (at 0 -3.85) (layer F.SilkS)
-      (effects (font (size 1 1) (thickness 0.15)))
-    )
+    (fp_text reference M3 (at -0.008 4.08) (layer F.SilkS)
+      (effects (font (size 1 1) (thickness 0.15)))
+    )
