File: sImCP.sch (KiCad schematic (older format))
At the start: 79 parts, among them J1 AVR-ISP-6, SW1 RESET, SW2 BOOT, U1 ATmega328P-AU, Y1 16MHz

Commit message: added new 3dmodels
Parts:
- gave numbers to parts that had none: 2
Changed lines of the file:
@@
 DOB1B
 $Comp
-L Mechanical:MountingHole H?
+L Mechanical:MountingHole H5
 U 1 1 60A7CB3E
 P 4150 7300
-F 0 "H?" H 4250 7346 50  0000 L CNN
+F 0 "H5" H 4250 7346 50  0000 L CNN
 F 1 "MountingHole" H 4250 7255 50  0000 L CNN
 F 2 "MountingHole:MountingHole_2.2mm_M2_DIN965_Pad" H 4150 7300 50  0001 C CNN
@@
 $EndComp
 $Comp
-L Mechanical:MountingHole H?
+L Mechanical:MountingHole H6
 U 1 1 60A7D760
 P 4850 7300
-F 0 "H?" H 4950 7346 50  0000 L CNN
+F 0 "H6" H 4950 7346 50  0000 L CNN
 F 1 "MountingHole" H 4950 7255 50  0000 L CNN
 F 2 "MountingHole:MountingHole_2.2mm_M2_DIN965_Pad" H 4850 7300 50  0001 C CNN

Commit message: update diode footprint to SOD-123FL
Parts:
- D1, D10, D11, D12, D13, D14, D15, D16, D17, D18, D19, D2, D20, D21, D3, D4, D5, D6, D7, D8, D9, DB1, DM1, DM2, DR1, DR2: footprint Diode_SMD:D_SOD-123F -> SOD-123FL:D_SOD-123FL
Changed lines of the file:
@@
 F 0 "D1" V 4696 1330 50  0000 R CNN
 F 1 "D_Small" V 4605 1330 50  0000 R CNN
-F 2 "Diode_SMD:D_SOD-123F" V 4650 1400 50  0001 C CNN
+F 2 "SOD-123FL:D_SOD-123FL" V 4650 1400 50  0001 C CNN
 F 3 "~" V 4650 1400 50  0001 C CNN
 F 4 "C426570" H 4650 1400 50  0001 C CNN "LCSC"
@@
 F 0 "D2" V 4696 2280 50  0000 R CNN
 F 1 "D_Small" V 4605 2280 50  0000 R CNN
-F 2 "Diode_SMD:D_SOD-123F" V 4650 2350 50  0001 C CNN
+F 2 "SOD-123FL:D_SOD-123FL" V 4650 2350 50  0001 C CNN
 F 3 "~" V 4650 2350 50  0001 C CNN
 F 4 "C426570" H 4650 2350 50  0001 C CNN "LCSC"
@@
 F 0 "D3" V 4696 2930 50  0000 R CNN
 F 1 "D_Small" V 4605 2930 50  0000 R CNN
-F 2 "Diode_SMD:D_SOD-123F" V 4650 3000 50  0001 C CNN
+F 2 "SOD-123FL:D_SOD-123FL" V 4650 3000 50  0001 C CNN
 F 3 "~" V 4650 3000 50  0001 C CNN
 F 4 "C426570" H 4650 3000 50  0001 C CNN "LCSC"
@@
 F 0 "D4" V 4696 3580 50  0000 R CNN
 F 1 "D_Small" V 4605 3580 50  0000 R CNN
-F 2 "Diode_SMD:D_SOD-123F" V 4650 3650 50  0001 C CNN
+F 2 "SOD-123FL:D_SOD-123FL" V 4650 3650 50  0001 C CNN
 F 3 "~" V 4650 3650 50  0001 C CNN
 F 4 "C426570" H 4650 3650 50  0001 C CNN "LCSC"
@@
 F 0 "D5" V 4696 4230 50  0000 R CNN
 F 1 "D_Small" V 4605 4230 50  0000 R CNN
-F 2 "Diode_SMD:D_SOD-123F" V 4650 4300 50  0001 C CNN
+F 2 "SOD-123FL:D_SOD-123FL" V 4650 4300 50  0001 C CNN
 F 3 "~" V 4650 4300 50  0001 C CNN
 F 4 "C426570" V 4650 4300 50  0001 C CNN "LCSC"
@@
 F 0 "D7" V 5296 2280 50  0000 R CNN
 F 1 "D_Small" V 5205 2280 50  0000 R CNN
-F 2 "Diode_SMD:D_SOD-123F" V 5250 2350 50  0001 C CNN
+F 2 "SOD-123FL:D_SOD-123FL" V 5250 2350 50  0001 C CNN
 F 3 "~" V 5250 2350 50  0001 C CNN
 F 4 "C426570" H 5250 2350 50  0001 C CNN "LCSC"
@@
 F 0 "D8" V 5296 2930 50  0000 R CNN
 F 1 "D_Small" V 5205 2930 50  0000 R CNN
-F 2 "Diode_SMD:D_SOD-123F" V 5250 3000 50  0001 C CNN
+F 2 "SOD-123FL:D_SOD-123FL" V 5250 3000 50  0001 C CNN
 F 3 "~" V 5250 3000 50  0001 C CNN
 F 4 "C426570" H 5250 3000 50  0001 C CNN "LCSC"
@@
 F 0 "D9" V 5296 3580 50  0000 R CNN
 F 1 "D_Small" V 5205 3580 50  0000 R CNN
-F 2 "Diode_SMD:D_SOD-123F" V 5250 3650 50  0001 C CNN
+F 2 "SOD-123FL:D_SOD-123FL" V 5250 3650 50  0001 C CNN
 F 3 "~" V 5250 3650 50  0001 C CNN
 F 4 "C426570" H 5250 3650 50  0001 C CNN "LCSC"
@@
 F 0 "D10" V 5296 4230 50  0000 R CNN
 F 1 "D_Small" V 5205 4230 50  0000 R CNN
-F 2 "Diode_SMD:D_SOD-123F" V 5250 4300 50  0001 C CNN
+F 2 "SOD-123FL:D_SOD-123FL" V 5250 4300 50  0001 C CNN
 F 3 "~" V 5250 4300 50  0001 C CNN
 F 4 "C426570" H 5250 4300 50  0001 C CNN "LCSC"
@@
 F 0 "D12" V 5896 2280 50  0000 R CNN
 F 1 "D_Small" V 5805 2280 50  0000 R CNN
-F 2 "Diode_SMD:D_SOD-123F" V 5850 2350 50  0001 C CNN
+F 2 "SOD-123FL:D_SOD-123FL" V 5850 2350 50  0001 C CNN
 F 3 "~" V 5850 2350 50  0001 C CNN
 F 4 "C426570" H 5850 2350 50  0001 C CNN "LCSC"
@@
 F 0 "D13" V 5896 2930 50  0000 R CNN
 F 1 "D_Small" V 5805 2930 50  0000 R CNN
-F 2 "Diode_SMD:D_SOD-123F" V 5850 3000 50  0001 C CNN
+F 2 "SOD-123FL:D_SOD-123FL" V 5850 3000 50  0001 C CNN
 F 3 "~" V 5850 3000 50  0001 C CNN
 F 4 "C426570" H 5850 3000 50  0001 C CNN "LCSC"
@@
 F 0 "D14" V 5896 3580 50  0000 R CNN
 F 1 "D_Small" V 5805 3580 50  0000 R CNN
-F 2 "Diode_SMD:D_SOD-123F" V 5850 3650 50  0001 C CNN
+F 2 "SOD-123FL:D_SOD-123FL" V 5850 3650 50  0001 C CNN
 F 3 "~" V 5850 3650 50  0001 C CNN
 F 4 "C426570" H 5850 3650 50  0001 C CNN "LCSC"
@@
 F 0 "D15" V 5896 4230 50  0000 R CNN
 F 1 "D_Small" V 5805 4230 50  0000 R CNN
-F 2 "Diode_SMD:D_SOD-123F" V 5850 4300 50  0001 C CNN
+F 2 "SOD-123FL:D_SOD-123FL" V 5850 4300 50  0001 C CNN
 F 3 "~" V 5850 4300 50  0001 C CNN
 F 4 "C426570" H 5850 4300 50  0001 C CNN "LCSC"
@@
 F 0 "D18" V 7196 2280 50  0000 R CNN
 F 1 "D_Small" V 7105 2280 50  0000 R CNN
-F 2 "Diode_SMD:D_SOD-123F" V 7150 2350 50  0001 C CNN
+F 2 "SOD-123FL:D_SOD-123FL" V 7150 2350 50  0001 C CNN
 F 3 "~" V 7150 2350 50  0001 C CNN
 F 4 "C426570" H 7150 2350 50  0001 C CNN "LCSC"
@@
 F 0 "D19" V 7196 2930 50  0000 R CNN
 F 1 "D_Small" V 7105 2930 50  0000 R CNN
-F 2 "Diode_SMD:D_SOD-123F" V 7150 3000 50  0001 C CNN
+F 2 "SOD-123FL:D_SOD-123FL" V 7150 3000 50  0001 C CNN
 F 3 "~" V 7150 3000 50  0001 C CNN
 F 4 "C426570" H 7150 3000 50  0001 C CNN "LCSC"
@@
 F 0 "D20" V 7196 3580 50  0000 R CNN
 F 1 "D_Small" V 7105 3580 50  0000 R CNN
-F 2 "Diode_SMD:D_SOD-123F" V 7150 3650 50  0001 C CNN
+F 2 "SOD-123FL:D_SOD-123FL" V 7150 3650 50  0001 C CNN
 F 3 "~" V 7150 3650 50  0001 C CNN
 F 4 "C426570" H 7150 3650 50  0001 C CNN "LCSC"
@@
 F 0 "D6" V 5296 1330 50  0000 R CNN
 F 1 "D_Small" V 5205 1330 50  0000 R CNN
-F 2 "Diode_SMD:D_SOD-123F" V 5250 1400 50  0001 C CNN
+F 2 "SOD-123FL:D_SOD-123FL" V 5250 1400 50  0001 C CNN
 F 3 "~" V 5250 1400 50  0001 C CNN
 F 4 "C426570" H 5250 1400 50  0001 C CNN "LCSC"
@@
 F 0 "D11" V 5896 1330 50  0000 R CNN
 F 1 "D_Small" V 5805 1330 50  0000 R CNN
-F 2 "Diode_SMD:D_SOD-123F" V 5850 1400 50  0001 C CNN
+F 2 "SOD-123FL:D_SOD-123FL" V 5850 1400 50  0001 C CNN
 F 3 "~" V 5850 1400 50  0001 C CNN
 F 4 "C426570" H 5850 1400 50  0001 C CNN "LCSC"
@@
 F 0 "D16" V 6496 1330 50  0000 R CNN
 F 1 "D_Small" V 6405 1330 50  0000 R CNN
-F 2 "Diode_SMD:D_SOD-123F" V 6450 1400 50  0001 C CNN
+F 2 "SOD-123FL:D_SOD-123FL" V 6450 1400 50  0001 C CNN
 F 3 "~" V 6450 1400 50  0001 C CNN
 F 4 "C426570" H 6450 1400 50  0001 C CNN "LCSC"
@@
 F 0 "DR1" V 6496 2280 50  0000 R CNN
 F 1 "D_Small" V 6405 2280 50  0000 R CNN
-F 2 "Diode_SMD:D_SOD-123F" V 6450 2350 50  0001 C CNN
+F 2 "SOD-123FL:D_SOD-123FL" V 6450 2350 50  0001 C CNN
 F 3 "~" V 6450 2350 50  0001 C CNN
 F 4 "C426570" H 6450 2350 50  0001 C CNN "LCSC"
@@
 F 0 "DR2" V 6496 2930 50  0000 R CNN
 F 1 "D_Small" V 6405 2930 50  0000 R CNN
-F 2 "Diode_SMD:D_SOD-123F" V 6450 3000 50  0001 C CNN
+F 2 "SOD-123FL:D_SOD-123FL" V 6450 3000 50  0001 C CNN
 F 3 "~" V 6450 3000 50  0001 C CNN
 F 4 "C426570" H 6450 3000 50  0001 C CNN "LCSC"
@@
 F 0 "DM1" V 6496 3580 50  0000 R CNN
 F 1 "D_Small" V 6405 3580 50  0000 R CNN
-F 2 "Diode_SMD:D_SOD-123F" V 6450 3650 50  0001 C CNN
+F 2 "SOD-123FL:D_SOD-123FL" V 6450 3650 50  0001 C CNN
 F 3 "~" V 6450 3650 50  0001 C CNN
 F 4 "C426570" H 6450 3650 50  0001 C CNN "LCSC"
@@
 F 0 "DM2" V 6496 4230 50  0000 R CNN
 F 1 "D_Small" V 6405 4230 50  0000 R CNN
-F 2 "Diode_SMD:D_SOD-123F" V 6450 4300 50  0001 C CNN
+F 2 "SOD-123FL:D_SOD-123FL" V 6450 4300 50  0001 C CNN
 F 3 "~" V 6450 4300 50  0001 C CNN
 F 4 "C426570" H 6450 4300 50  0001 C CNN "LCSC"
@@
 F 0 "D17" V 7196 1330 50  0000 R CNN
 F 1 "D_Small" V 7105 1330 50  0000 R CNN
-F 2 "Diode_SMD:D_SOD-123F" V 7150 1400 50  0001 C CNN
+F 2 "SOD-123FL:D_SOD-123FL" V 7150 1400 50  0001 C CNN
 F 3 "~" V 7150 1400 50  0001 C CNN
 F 4 "C426570" H 7150 1400 50  0001 C CNN "LCSC"
@@
 F 0 "D21" V 7196 4230 50  0000 R CNN
 F 1 "D_Small" V 7105 4230 50  0000 R CNN
-F 2 "Diode_SMD:D_SOD-123F" V 7150 4300 50  0001 C CNN
+F 2 "SOD-123FL:D_SOD-123FL" V 7150 4300 50  0001 C CNN
 F 3 "~" V 7150 4300 50  0001 C CNN
 F 4 "C426570" H 7150 4300 50  0001 C CNN "LCSC"
@@
 F 0 "DB1" H 4500 4800 50  0000 R CNN
 F 1 "D_Small" H 4700 4700 50  0000 R CNN
-F 2 "Diode_SMD:D_SOD-123F" V 4450 4900 50  0001 C CNN
+F 2 "SOD-123FL:D_SOD-123FL" V 4450 4900 50  0001 C CNN
 F 3 "~" V 4450 4900 50  0001 C CNN
 F 4 "C426570" H 4450 4900 50  0001 C CNN "LCSC"
