File: PCB/sImCP.sch (KiCad schematic (older format))
At the start: 79 parts, among them J1 AVR-ISP-6, SW1 RESET, SW2 BOOT, U1 ATmega328P-AU, Y1 16MHz

Commit message: [FAB FILES] feat: changed 4u7 capacitor to THT
Changed capacitor to THT as previous part number has no stock
Regenerated fabrication files
Parts:
- C5: footprint Capacitor_SMD:CP_Elec_4x5.3 -> Capacitor_THT:CP_Radial_D4.0mm_P1.50mm; LCSC C134741 -> C47879
Changed lines of the file:
@@
 F 0 "C5" H 3241 4846 50  0000 L CNN
 F 1 "4.7uF" H 3241 4755 50  0000 L CNN
-F 2 "Capacitor_SMD:CP_Elec_4x5.3" H 3150 4800 50  0001 C CNN
+F 2 "Capacitor_THT:CP_Radial_D4.0mm_P1.50mm" H 3150 4800 50  0001 C CNN
 F 3 "~" H 3150 4800 50  0001 C CNN
-F 4 "C134741" H 3150 4800 50  0001 C CNN "LCSC"
+F 4 "C47879" H 3150 4800 50  0001 C CNN "LCSC"
 	1    3150 4800
 	1    0    0    -1
